Commit message: .

File: polydog.urdf (robot description, URDF)
Before this commit: robot robot_dog, 18 links, 17 joints
Joints:
- removed joint hip1
- removed joint hip2
- removed joint hip3
- removed joint hip4
- removed joint knee1
- removed joint knee2
- removed joint knee3
- removed joint knee4
- removed joint shoulder1
- removed joint shoulder2
- removed joint shoulder3
- removed joint shoulder4
- added joint FL1_joint: type revolute, parent body, child case2, origin xyz=0.084 -0.122 0 rpy=1.5708 0 0, axis 0 0 1, limit lower=-3 upper=3 effort=10 velocity=6
- added joint FL2_joint: type revolute, parent case2, child femur2, origin xyz=0.035 0 0.018 rpy=3.14 3.14 0, axis 1 0 0, limit lower=-3 upper=3 effort=10 velocity=6
- added joint FL3_joint: type revolute, parent femur2, child tibia2, origin xyz=-0.0075 0.129 0.0015 rpy=1.57 0 0, axis 1 0 0, limit lower=-3 upper=3 effort=10 velocity=6
- added joint FR1_joint: type revolute, parent body, child case3, origin xyz=-0.084 -0.122 0 rpy=1.5708 0 3.14, axis 0 0 1, limit lower=-3 upper=3 effort=10 velocity=6
- added joint FR2_joint: type revolute, parent case3, child femur3, origin xyz=0.035 0 -0.018 rpy=3.14 3.14 0, axis 1 0 0, limit lower=-3 upper=3 effort=10 velocity=6
- added joint FR3_joint: type revolute, parent femur3, child tibia3, origin xyz=-0.0075 0.129 0.0015 rpy=1.57 3.14 0, axis 1 0 0, limit lower=-3 upper=3 effort=10 velocity=6
- added joint RL1_joint: type revolute, parent body, child case1, origin xyz=0.084 0.122 0 rpy=1.5708 0 0, axis 0 0 1, limit lower=-3 upper=+3 effort=10 velocity=6
- added joint RL2_joint: type revolute, parent case1, child femur1, origin xyz=0.035 0 -0.018 rpy=-3.14 3.14 0, axis 1 0 0, limit lower=-3 upper=3 effort=10 velocity=6
- added joint RL3_joint: type revolute, parent femur1, child tibia1, origin xyz=-0.0075 0.129 0.0015 rpy=1.57 0 0, axis 1 0 0, limit lower=-3 upper=3 effort=10 velocity=6
- added joint RR1_joint: type revolute, parent body, child case4, origin xyz=-0.084 0.122 0 rpy=1.5708 0 3.14, axis 0 0 1, limit lower=-3 upper=3 effort=10 velocity=6
- added joint RR2_joint: type revolute, parent case4, child femur4, origin xyz=0.035 0 0.018 rpy=3.14 3.14 0, axis 1 0 0, limit lower=-3 upper=3 effort=10 velocity=6
- added joint RR3_joint: type revolute, parent femur4, child tibia4, origin xyz=-0.0075 0.129 0.0015 rpy=1.57 3.14 0, axis 1 0 0, limit lower=-3 upper=3 effort=10 velocity=6
