Commit message: .

File: src/polydog_description/urdf/polydog.urdf (robot description, URDF)
Before this commit: robot polydog, 18 links, 17 joints
Links:
- added link depth_camera_link, mass 1e-5; collision box size=0.0235 0.08 0.015; visual box size=0.0235 0.08 0.015
- added link imu_sensor_link, mass 0.001; collision box size=0.02 0.02 0.02; visual box size=0.02 0.02 0.02
Joints:
- added joint depth_camera_joint: type fixed, parent body, child depth_camera_link, origin xyz=0 -0.197 0.0265 rpy=0 0 -1.57, axis 0 0 0
- added joint imu_sensor_joint: type fixed, parent body, child imu_sensor_link, origin xyz=0 0 0 rpy=0 0 0, axis 0 0 0
